File: ki_cad/soundseeker/piezo_driver.kicad_sch (KiCad schematic)
At the start: 1 part

Commit message: add preamp schematic
Parts:
- removed U?: OPA453, Package_TO_SOT_SMD:TO-263-7_TabPin4, symbol soundseeker:OPA453
Changed lines of the file:
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@@
 (kicad_sch (version 20211123) (generator eeschema)
   (paper "A4")
-  (wire (pts (xy 111.76 101.6) (xy 111.76 102.87))
-    (stroke (width 0) (type default) (color 0 0 0 0))
-  )
-  (symbol (lib_id "power:GND") (at 111.76 102.87 0) (unit 1)
-    (in_bom yes) (on_board yes) (fields_autoplaced)
-    (property "Reference" "#PWR0115" (id 0) (at 111.76 109.22 0)
-      (effects (font (size 1.27 1.27)) hide)
-    )
-    (property "Value" "GND" (id 1) (at 111.76 107.95 0))
-    (property "Footprint" "" (id 2) (at 111.76 102.87 0)
-      (effects (font (size 1.27 1.27)) hide)
-    )
-    (property "Datasheet" "" (id 3) (at 111.76 102.87 0)
-      (effects (font (size 1.27 1.27)) hide)
-    )
-    (pin "1")
-  )
-  (symbol (lib_id "soundseeker:OPA453") (at 114.3 93.98 0) (unit 1)
-    (in_bom yes) (on_board yes) (fields_autoplaced)
-    (property "Reference" "U?" (id 0) (at 124.46 89.281 0))
-    (property "Value" "OPA453" (id 1) (at 124.46 91.821 0))
-    (property "Footprint" "Package_TO_SOT_SMD:TO-263-7_TabPin4" (id 2) (at 137.16 97.79 0)
-      (effects (font (size 1.27 1.27)) hide)
-    )
-    (property "Datasheet" "https://www.ti.com/lit/ds/symlink/opa453.pdf" (id 3) (at 139.7 100.33 0)
-      (effects (font (size 1.27 1.27)) hide)
-    )
-    (pin "1")
-    (pin "2")
-    (pin "4")
-    (pin "5")
-    (pin "6")
-    (pin "7")
-  )
 )
