File: ki_cad/soundseeker/high_voltage_power_supply.kicad_sch (KiCad schematic)
At the start: 34 parts

Commit message: schematic
Parts:
- removed C?: 1u, Capacitor_SMD:C_1206_3216Metric_Pad1.33x1.80mm_HandSolder, symbol Device:C
- removed R?: 750, Resistor_SMD:R_0805_2012Metric_Pad1.20x1.40mm_HandSolder, symbol Device:R
- removed R?: 47k, Resistor_SMD:R_0805_2012Metric_Pad1.20x1.40mm_HandSolder, symbol Device:R
- removed R?: 10k, Resistor_SMD:R_0805_2012Metric_Pad1.20x1.40mm_HandSolder, symbol Device:R
- removed U?: TLV9052S, Package_SO:MSOP-10_3x3mm_P0.5mm, symbol soundseeker:TLV9052S
- added C?: 10n, Resistor_SMD:R_0805_2012Metric_Pad1.20x1.40mm_HandSolder, symbol Device:C
- added C?: 470p, Resistor_SMD:R_0805_2012Metric_Pad1.20x1.40mm_HandSolder, symbol Device:C
- added C? (x2): 1u, Capacitor_SMD:C_1206_3216Metric_Pad1.33x1.80mm_HandSolder, symbol Device:C
- added J?: Conn_01x11, symbol Connector_Generic:Conn_01x11
- added R? (x7): 2k, Resistor_SMD:R_0805_2012Metric_Pad1.20x1.40mm_HandSolder, symbol Device:R
- added R? (x5): 1k, Resistor_SMD:R_0805_2012Metric_Pad1.20x1.40mm_HandSolder, symbol Device:R
- C?: value 1u -> 10n
- R?: value 100k -> 47k
- R?: value 10k -> 1k
- R?: value 1.5k -> 100
- R?: value 3.3k -> 2.2k
- R?: value 20k -> 2.2k
Connections:
- net vgnd_pwm_opa is gone; now on an unnamed net: R?.1
- net +5V: now also C?.1, C?.1, C?.1, L?.1, U?.3 (CS), U?.8 (Vin), J?.11 (Pin_11)
- net GND: now also C?.2, C?.2, J?.10 (Pin_10), J?.2 (Pin_2), R?.2
- net V_piezo_drive: now also C?.1, C?.1
- net enable_piezo_driver: now also J?.9 (Pin_9)
- net vref_power_opa: now also U?.1 (+); no longer R?.1
- net piezo_out: now reaches C?.2, R?.2, U?.6
- net piezo_out: now also J?.1 (Pin_1)
- net at R?.2, U?.1: now also C?.1, C?.2
- net vref_preamp: now reaches C?.1, R?.1, R?.2
- net vref_preamp: now also U?.3 (+)
- net at R?.1, R?.2, U?.2 (-): now also C?.1
- net at C?.2: no longer U?.3 (+)
- net pwm_signal_in: no longer names the net of R?.1
- net pwm_signal_in: now also R?.1, R?.2
- new net: C?.2, R?.1
- new net: R?.1, R?.1, R?.2 (x4)
- new net: R?.1, R?.1, R?.1
- new net dac_in_1_lsb: J?.3 (Pin_3), R?.2
- new net dac_in_2: J?.4 (Pin_4), R?.2
- new net dac_in_3: J?.5 (Pin_5), R?.2
- new net dac_in_4: J?.6 (Pin_6), R?.2
- new net dac_in_5: J?.7 (Pin_7), R?.2
- new net dac_in_6_msb: J?.8 (Pin_8), R?.2
Other:
- moved on the sheet: C?, D?, L?, Q?, R?, U?, U?A, U?C

Commit message: add preamp schematic
Parts:
- added C16: 1u, Resistor_SMD:R_0805_2012Metric_Pad1.20x1.40mm_HandSolder, symbol Device:C
- added R?: 15k, Resistor_SMD:R_0805_2012Metric_Pad1.20x1.40mm_HandSolder, symbol Device:R
- C3: renamed from C?; value 100n -> 1u; footprint Resistor_SMD:R_1206_3216Metric_Pad1.30x1.75mm_HandSolder -> Resistor_SMD:R_0805_2012Metric_Pad1.20x1.40mm_HandSolder
- C5: renamed from C?; footprint (none) -> Capacitor_SMD:C_0805_2012Metric_Pad1.18x1.45mm_HandSolder
- J1: renamed from J?; footprint (none) -> Connector_PinHeader_2.54mm:PinHeader_1x11_P2.54mm_Vertical
- R15: renamed from R?; value 100k -> 56k
- gave numbers to parts that had none: 41
Connections:
- net +5V: now also C16.1
- net GND: now also C16.2
Other:
- moved on the sheet: U2C

Commit message: add buttons and display spi connections
Parts:
- removed C10: 470p, Resistor_SMD:R_0805_2012Metric_Pad1.20x1.40mm_HandSolder, symbol Device:C
- removed C16: 1u, Resistor_SMD:R_0805_2012Metric_Pad1.20x1.40mm_HandSolder, symbol Device:C
- removed C4: 10u, Resistor_SMD:R_1206_3216Metric_Pad1.30x1.75mm_HandSolder, symbol Device:C
- removed C7: 10n, Resistor_SMD:R_0805_2012Metric_Pad1.20x1.40mm_HandSolder, symbol Device:C
- removed R13, R14: 20k, Resistor_SMD:R_0805_2012Metric_Pad1.20x1.40mm_HandSolder, symbol Device:R
- removed R18: 1k, Resistor_SMD:R_0805_2012Metric_Pad1.20x1.40mm_HandSolder, symbol Device:R
- removed R19: 2.2k, Resistor_SMD:R_0805_2012Metric_Pad1.20x1.40mm_HandSolder, symbol Device:R
- removed R?: 15k, Resistor_SMD:R_0805_2012Metric_Pad1.20x1.40mm_HandSolder, symbol Device:R
- removed U2: TLV9052S, Package_SO:MSOP-10_3x3mm_P0.5mm, symbol soundseeker:TLV9052S
- removed U3: OPA453, Package_TO_SOT_SMD:TO-263-7_TabPin4, symbol soundseeker:OPA453
- added U? (x3): MC34072, Package_SO:SOIC-8_3.9x4.9mm_P1.27mm, symbol soundseeker:MC34072
- C13: value 15p -> 68p
- L1: value 2.2u -> 3.3u
- R20: value 2.2k -> 1.69k
- R21: value 47k -> 22k
Connections:
- net GND: now also C14.1, C15.1, U?.4 (V-); no longer C14.2, C15.2
- net V_piezo_drive: now also C14.2, U?.8 (V+); no longer C14.1
- net piezo_out: now also C13.1, R21.1, U?.7; no longer C13.2, R21.2
- net vref_power_opa: now also U?.1, U?.2 (-), U?.5 (+); no longer C15.1, R22.2, R23.1
- net at C12.1: now also C5.1, R17.2
- new net: C13.2, R20.2, R21.2, U?.6 (-)
- new net: C15.2, R22.2, R23.1, U?.3 (+)
Other:
- moved on the sheet: C12, C13, C14, C15, R20, R21, R22, R23

Commit message: sounseeker base board (evaluartion) PCB layout
Parts:
- removed C6: 1u, Capacitor_SMD:C_1206_3216Metric_Pad1.33x1.80mm_HandSolder, symbol Device:C
- removed J1: Conn_01x11, Connector_PinHeader_2.54mm:PinHeader_1x11_P2.54mm_Vertical, symbol Connector_Generic:Conn_01x11
- added J1: Piezo Driver Out, Connector_PinHeader_2.54mm:PinHeader_1x02_P2.54mm_Vertical, symbol Connector_Generic:Conn_01x02
- gave numbers to parts that had none: 1
Connections:
- net GND: now also J1.2 (Pin_2)
- net piezo_out: no longer names the net of C13.1, R21.1, U3.7
- net piezo_out: now also J1.1 (Pin_1)
Other:
- moved on the sheet: C11, C15, C8, C9, R22, R23, U3A

Commit message: finish base board (evaluation)
Parts:
- C1, C2: footprint Resistor_SMD:R_1206_3216Metric_Pad1.30x1.75mm_HandSolder -> Capacitor_SMD:C_1206_3216Metric_Pad1.33x1.80mm_HandSolder
- C12, C13, C3: footprint Resistor_SMD:R_0805_2012Metric_Pad1.20x1.40mm_HandSolder -> Capacitor_SMD:C_0805_2012Metric_Pad1.18x1.45mm_HandSolder
- D1: footprint Diode_SMD:D_SOD-128 -> Diode_SMD:D_SMA
- J1: value Piezo Driver Out -> 1x02; description (none) -> PIEZO_OUT
Changed lines of the file:
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@@
     (property "Reference" "C12" (id 0) (at 149.86 110.49 90))
     (property "Value" "10n" (id 1) (at 149.86 113.03 90))
-    (property "Footprint" "Resistor_SMD:R_0805_2012Metric_Pad1.20x1.40mm_HandSolder" (id 2) (at 153.67 118.4148 0)
+    (property "Footprint" "Capacitor_SMD:C_0805_2012Metric_Pad1.18x1.45mm_HandSolder" (id 2) (at 153.67 118.4148 0)
       (effects (font (size 1.27 1.27)) hide)
     )
@@
     (property "Reference" "D1" (id 0) (at 122.2375 39.37 0))
     (property "Value" "RB058L150DDTE25" (id 1) (at 122.2375 41.91 0))
-    (property "Footprint" "Diode_SMD:D_SOD-128" (id 2) (at 121.92 45.72 0)
+    (property "Footprint" "Diode_SMD:D_SMA" (id 2) (at 121.92 45.72 0)
       (effects (font (size 1.27 1.27)) hide)
     )
@@
       (effects (font (size 1.27 1.27)) (justify left))
     )
-    (property "Footprint" "Resistor_SMD:R_0805_2012Metric_Pad1.20x1.40mm_HandSolder" (id 2) (at 50.4952 53.34 0)
+    (property "Footprint" "Capacitor_SMD:C_0805_2012Metric_Pad1.18x1.45mm_HandSolder" (id 2) (at 50.4952 53.34 0)
       (effects (font (size 1.27 1.27)) hide)
     )
@@
   )
   (symbol (lib_id "Connector_Generic:Conn_01x02") (at 204.47 116.84 0) (unit 1)
-    (in_bom yes) (on_board yes) (fields_autoplaced)
+    (in_bom yes) (on_board yes)
     (property "Reference" "J1" (id 0) (at 207.01 116.8399 0)
       (effects (font (size 1.27 1.27)) (justify left))
     )
-    (property "Value" "Piezo Driver Out" (id 1) (at 207.01 119.3799 0)
+    (property "Value" "1x02" (id 1) (at 207.01 119.3799 0)
       (effects (font (size 1.27 1.27)) (justify left))
     )
@@
       (effects (font (size 1.27 1.27)) hide)
     )
+    (property "description" "PIEZO_OUT" (id 4) (at 205.74 121.92 0))
     (pin "1")
     (pin "2")
@@
     (property "Reference" "C13" (id 0) (at 182.88 147.32 90))
     (property "Value" "68p" (id 1) (at 182.88 144.78 90))
-    (property "Footprint" "Resistor_SMD:R_0805_2012Metric_Pad1.20x1.40mm_HandSolder" (id 2) (at 179.07 141.9352 0)
+    (property "Footprint" "Capacitor_SMD:C_0805_2012Metric_Pad1.18x1.45mm_HandSolder" (id 2) (at 179.07 141.9352 0)
       (effects (font (size 1.27 1.27)) hide)
     )
@@
       (effects (font (size 1.27 1.27)) (justify left))
     )
-    (property "Footprint" "Resistor_SMD:R_1206_3216Metric_Pad1.30x1.75mm_HandSolder" (id 2) (at 27.6352 53.34 0)
+    (property "Footprint" "Capacitor_SMD:C_1206_3216Metric_Pad1.33x1.80mm_HandSolder" (id 2) (at 27.6352 53.34 0)
       (effects (font (size 1.27 1.27)) hide)
     )
@@
       (effects (font (size 1.27 1.27)) (justify left))
     )
-    (property "Footprint" "Resistor_SMD:R_1206_3216Metric_Pad1.30x1.75mm_HandSolder" (id 2) (at 39.0652 53.34 0)
-      (effects (font (size 1.27 1.27)) hide)
-    )
+    (property "Footprint" "Capacitor_SMD:C_1206_3216Metric_Pad1.33x1.80mm_HandSolder" (id 2) (at 39.0652 53.34 0)
+      (effects (font (size 1.27 1.27)) hide)
+    )

Commit message: first working hardware board :)
Parts:
- C13: value 68p -> 15p
- R20: value 1.69k -> 10k
- R21: value 22k -> 150k
Changed lines of the file:
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@@
       (effects (font (size 1.27 1.27)) (justify left))
     )
-    (property "Value" "22k" (id 1) (at 181.61 130.81 90)
+    (property "Value" "150k" (id 1) (at 181.61 130.81 90)
       (effects (font (size 1.27 1.27)) (justify left))
     )
@@
   (symbol (lib_id "Device:R") (at 163.83 119.38 90) (unit 1)
     (in_bom yes) (on_board yes)
-    (property "Reference" "R20" (id 0) (at 163.83 111.76 90)
-      (effects (font (size 1.27 1.27)) (justify left))
-    )
-    (property "Value" "1.69k" (id 1) (at 165.1 114.3 90)
+    (property "Reference" "R20" (id 0) (at 165.1 111.76 90)
+      (effects (font (size 1.27 1.27)) (justify left))
+    )
+    (property "Value" "10k" (id 1) (at 165.1 114.3 90)
       (effects (font (size 1.27 1.27)) (justify left))
     )
@@
     (in_bom yes) (on_board yes)
     (property "Reference" "C13" (id 0) (at 182.88 147.32 90))
-    (property "Value" "68p" (id 1) (at 182.88 144.78 90))
+    (property "Value" "15p" (id 1) (at 182.88 144.78 90))
     (property "Footprint" "Capacitor_SMD:C_0805_2012Metric_Pad1.18x1.45mm_HandSolder" (id 2) (at 179.07 141.9352 0)
       (effects (font (size 1.27 1.27)) hide)
