File: ki_cad/soundseeker/soundseeker.kicad_pcb (KiCad board)
At the start: 2 copper layers, 85.4 x 59 mm, 80 parts, among them J1 Piezo Driver Out, J2 TFT_DISPLAY, J3 UART, J4 SWD, J5 preamp_in, J6 x10, J7 x20, J8 x2, Q1 FDT86113LZ, SW1 SW_LEFT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

Commit message: finish base board (evaluation)
Parts:
- removed REF** (x4): MountingHole_2mm, MountingHole:MountingHole_2mm
- C1, C2, C20, C21: footprint Resistor_SMD:R_1206_3216Metric_Pad1.30x1.75mm_HandSolder -> Capacitor_SMD:C_1206_3216Metric_Pad1.33x1.80mm_HandSolder
- C10, C12, C13, C19, C22, C3, C4: footprint Resistor_SMD:R_0805_2012Metric_Pad1.20x1.40mm_HandSolder -> Capacitor_SMD:C_0805_2012Metric_Pad1.18x1.45mm_HandSolder
- D1: value RB058L150DDTE25 -> SS 16 VIS; footprint Diode_SMD:D_SOD-128 -> Diode_SMD:D_SMA
- J1: value Piezo Driver Out -> 1x02
- J2: value TFT_DISPLAY -> 1x08
- J3: value UART -> 1x03
- J4: value SWD -> 1x03
- J5: value preamp_in -> 1x03
- J6: value x10 -> 1x02
- J7: value x20 -> 1x02
- J8: value x2 -> 1x02
- SW1: value SW_LEFT -> SW
- SW2: value SW_RIGHT -> SW
- SW3: value SW_UP -> SW
- SW4: value SW_DOWN -> SW
- SW5: value SW_BACK -> SW
- SW6: value SW_OK -> SW
Routing:
- net GND: vias 53 -> 52
Other:
- outline, holes or cut-outs redrawn
- board text added: "piezo_out"
- board text added: "preamp_in"

Commit message: first working hardware board :)
Parts:
- C13: value 68p -> 15p
- D1: value SS 16 VIS -> RB058L150DDTE25
- R20: value 1.69k -> 10k
- R21: value 22k -> 150k
